File: pcb/hajken_cutouts/smartcar_shield_cutouts.brd (EAGLE design)
At the start: 87.8 x 96.4 mm, 14 parts, among them J1 ARDUINO_R3_SHIELDUNO_R3_SHIEL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

Commit message: Subject: Update PCB board - ready for production
Co-authored-by: JonatanVaara <jonatan.vaara94@gmail.com>
Co-authored-by: EmanuelDellsen <emanuel.dellsen@gmail.com>
Co-authored-by: strand93 <strand.93@hotmail.com>
Co-authored-by: NiklasMoller <niklasxmoller@gmail.com>
Co-authored-by: KarlWestgardh <karl.westgardh@gmail.com>
Parts:
- moved SERIAL_2 10.9 mm to (-22.9, 14.0), turned to 90 degrees
- renumbered DRIVING to DRIVING_ON_ROUTE
Routing:
- net RX_BLUE: track 77.8 -> 72.0 mm
- net GND: track 252.8 -> 258.5 mm
- net TX_BLUE: track 90.1 -> 92.1 mm
Other:
- outline, holes or cut-outs redrawn
- board text added: "DIT112 - VT19"
- board text added: "RX"
- board text added: "TX"
- board text added: "_-_- _/\______\\__ _-_-__ / ,-. -|- ,-.`-. _-_ _-_- `( o )----( o )-' `-' `-'"
- board text added: "_-_- _/|______\\__ _-_-__ / ,-. -|- ,-.`-. _-_- `( o )----( o )-' `-' `-' You draw, we drive!"
- board text removed: "_-_- _/\______\\__ _-_-__ / ,-. -|- ,-.`-. _-_- `( o )----( o )-' `-' `-' You draw, we drive!"
